File: KiCad/Stormbreaker.kicad_sch (KiCad schematic)
At the start: 37 parts, among them J1 Micro_SD_Card_Det2, Q2 PMOS, SW1 SW_Push, U1 BQ25895RTW, U3 ATtiny1616-M

Commit message: I am suffering
Parts:
- BT1: footprint (none) -> Connector_JST:JST_PH_B2B-PH-K_1x02_P2.00mm_Vertical
- C1, C13, C2, C3, C4, C5, C6, C7: footprint (none) -> Capacitor_SMD:C_0603_1608Metric
- C10, C12, C8: footprint Capacitor_SMD:C_0402_1005Metric -> Capacitor_SMD:C_0603_1608Metric
- R1, R10, R2, R3, R4, R5, R6, R7, R8, R9: footprint (none) -> Resistor_SMD:R_0603_1608Metric
- SW1: footprint (none) -> Button_Switch_THT:SW_Tactile_SPST_Angled_PTS645Vx39-2LFS
Changed lines of the file:
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@@
 			)
 		)
-		(property "Footprint" "Capacitor_SMD:C_0402_1005Metric"
+		(property "Footprint" "Capacitor_SMD:C_0603_1608Metric"
 			(at 45.72 156.21 0)
 			(effects
@@
 			)
 		)
-		(property "Footprint" ""
+		(property "Footprint" "Connector_JST:JST_PH_B2B-PH-K_1x02_P2.00mm_Vertical"
 			(at 114.3 87.376 90)
 			(effects
@@
 			)
 		)
-		(property "Footprint" "Capacitor_SMD:C_0402_1005Metric"
+		(property "Footprint" "Capacitor_SMD:C_0603_1608Metric"
 			(at 62.23 160.02 0)
 			(effects
@@
 			)
 		)
-		(property "Footprint" "Capacitor_SMD:C_0402_1005Metric"
+		(property "Footprint" "Capacitor_SMD:C_0603_1608Metric"
 			(at 148.59 156.21 0)
 			(effects
@@
 			)
 		)
-		(property "Footprint" ""
+		(property "Footprint" "Button_Switch_THT:SW_Tactile_SPST_Angled_PTS645Vx39-2LFS"
 			(at 210.82 69.85 0)
 			(effects
@@
 			)
 		)
-		(property "Footprint" ""
+		(property "Footprint" "Resistor_SMD:R_0603_1608Metric"
 			(at 97.79 104.14 0)
 			(effects
@@
 			)
 		)
-		(property "Footprint" ""
+		(property "Footprint" "Capacitor_SMD:C_0603_1608Metric"
 			(at 109.22 95.25 0)
 			(effects
@@
 			)
 		)
-		(property "Footprint" ""
+		(property "Footprint" "Capacitor_SMD:C_0603_1608Metric"
 			(at 71.12 68.58 0)
 			(effects
@@
 			)
 		)
-		(property "Footprint" ""
+		(property "Footprint" "Resistor_SMD:R_0603_1608Metric"
 			(at 58.42 71.12 0)
 			(effects
@@
 			)
 		)
-		(property "Footprint" ""
+		(property "Footprint" "Capacitor_SMD:C_0603_1608Metric"
 			(at 125.73 73.66 0)
 			(effects
@@
 			)
 		)
-		(property "Footprint" ""
+		(property "Footprint" "Resistor_SMD:R_0603_1608Metric"
 			(at 193.04 72.39 0)
 			(effects
@@
 			)
 		)
-		(property "Footprint" ""
+		(property "Footprint" "Resistor_SMD:R_0603_1608Metric"
 			(at 73.66 78.74 0)
 			(effects
@@
 			)
 		)
-		(property "Footprint" ""
+		(property "Footprint" "Resistor_SMD:R_0603_1608Metric"
 			(at 199.39 88.9 0)
 			(effects
@@
 			)
 		)
-		(property "Footprint" ""
+		(property "Footprint" "Capacitor_SMD:C_0603_1608Metric"
 			(at 116.84 73.66 0)
 			(effects
@@
 			)
 		)
-		(property "Footprint" ""
+		(property "Footprint" "Capacitor_SMD:C_0603_1608Metric"
 			(at 109.22 87.63 0)
 			(effects
@@
 			)
 		)
-		(property "Footprint" ""
+		(property "Footprint" "Resistor_SMD:R_0603_1608Metric"
 			(at 135.89 93.98 0)
 			(effects
@@
 			)
 		)
-		(property "Footprint" ""
+		(property "Footprint" "Resistor_SMD:R_0603_1608Metric"
 			(at 182.88 60.96 0)
 			(effects
@@
 			)
 		)
-		(property "Footprint" ""
+		(property "Footprint" "Capacitor_SMD:C_0603_1608Metric"
 			(at 99.06 74.93 0)
 			(effects
@@
 			)
 		)
-		(property "Footprint" ""
+		(property "Footprint" "Resistor_SMD:R_0603_1608Metric"
 			(at 97.79 99.06 0)
 			(effects
@@
 			)
 		)
-		(property "Footprint" ""
+		(property "Footprint" "Capacitor_SMD:C_0603_1608Metric"
 			(at 162.56 53.34 0)
 			(effects
@@
 			)
 		)
-		(property "Footprint" ""
+		(property "Footprint" "Resistor_SMD:R_0603_1608Metric"
 			(at 143.51 93.98 0)
 			(effects
@@
 			)
 		)
-		(property "Footprint" ""
+		(property "Footprint" "Capacitor_SMD:C_0603_1608Metric"
 			(at 110.49 66.04 0)
 			(effects
@@
 			)
 		)
-		(property "Footprint" ""
+		(property "Footprint" "Resistor_SMD:R_0603_1608Metric"
 			(at 191.77 88.9 0)
 			(effects

Commit message: aaaaaaaaa
Parts:
- added BT2: Battery_Cell, Connector_JST:JST_PH_B2B-PH-K_1x02_P2.00mm_Vertical, symbol Device:Battery_Cell
Connections:
- net GND: now also BT2.2 (-)
- net at BT1.1 (+), C2.1, U1.13 (BAT)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: now also BT2.1 (+)
Changed lines of the file:
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@@
 	)
 	(junction
+		(at 114.3 83.82)
+		(diameter 0)
+		(color 0 0 0 0)
+	)
+	(junction
 		(at 99.06 71.12)
 		(diameter 0)
@@
 	(wire
 		(pts
+			(xy 114.3 83.82) (xy 124.46 83.82)
+		)
+		(stroke
+			(width 0)
+			(type default)
+		)
+	)
+	(wire
+		(pts
 			(xy 154.94 54.61) (xy 154.94 53.34)
 		)
@@
 	(wire
 		(pts
+			(xy 114.3 91.44) (xy 124.46 91.44)
+		)
+		(stroke
+			(width 0)
+			(type default)
+		)
+	)
+	(wire
+		(pts
 			(xy 62.23 147.32) (xy 62.23 156.21)
 		)
@@
 				)
 				(justify left)
+				(hide yes)
 			)
 		)
@@
 					(unit 1)
 				)
+			)
+		)
+	)
+	(symbol
+		(lib_id "Device:Battery_Cell")
+		(at 124.46 88.9 0)
+		(unit 1)
+		(exclude_from_sim no)
+		(in_bom yes)
+		(on_board yes)
+		(dnp no)
+		(fields_autoplaced yes)
+		(property "Reference" "BT2"
+			(at 128.27 85.7884 0)
+			(effects
+				(font
+					(size 1.27 1.27)
+				)
+				(justify left)
+			)
+		)
+		(property "Value" "Battery_Cell"
+			(at 128.27 88.3284 0)
+			(effects
+				(font
+					(size 1.27 1.27)
+				)
+				(justify left)
+				(hide yes)
+			)
+		)
+		(property "Footprint" "Connector_JST:JST_PH_B2B-PH-K_1x02_P2.00mm_Vertical"
+			(at 124.46 87.376 90)
+			(effects
+				(font
+					(size 1.27 1.27)
+				)
+				(hide yes)
+			)
+		)
+		(property "Datasheet" "~"
+			(at 124.46 87.376 90)
+			(effects
+				(font
+					(size 1.27 1.27)
+				)
+				(hide yes)
+			)
+		)
+		(property "Description" "Single-cell battery"
+			(at 124.46 88.9 0)
+			(effects
+				(font
+					(size 1.27 1.27)
+				)
+				(hide yes)
+			)
+		)
+		(pin "2"
+		)
+		(pin "1"
+		)
+		(instances
+			(project "Stormbreaker"
+				(path "/dcc89f95-4ae4-4756-aa81-33bf4d3c86ca"
+					(reference "BT2")
+					(unit 1)
+				)

Commit message: Stuff
Parts:
- added J2: USB_C_Receptacle, Connector_USB:USB_C_Receptacle_Amphenol_12401548E4-2A, symbol Connector:USB_C_Receptacle
- added J3: 505278-1933, Stormbreaker:5052781933, symbol SamacSys_Parts:505278-1933
- added Q2, Q3: PMOS, symbol Simulation_SPICE:PMOS
- added R11, R12: 10k, Resistor_SMD:R_0402_1005Metric, symbol Device:R_Small
- added R13, R14: 100k, Resistor_SMD:R_0603_1608Metric, symbol Device:R_Small
- added TP10: 3V3_OUT, TestPoint:TestPoint_Pad_D1.5mm, symbol Connector:TestPoint
- added TP6: POWER, TestPoint:TestPoint_Pad_D1.5mm, symbol Connector:TestPoint
- added TP7: SHUTDOWN, TestPoint:TestPoint_Pad_D1.5mm, symbol Connector:TestPoint
- added TP8: 1V8_IN, TestPoint:TestPoint_Pad_D1.5mm, symbol Connector:TestPoint
- added TP9: 1V8_OUT, TestPoint:TestPoint_Pad_D1.5mm, symbol Connector:TestPoint
- added U4: ~, Stormbreaker:melonHD_SMT, symbol melonHD_module:melonHD_SMT
- renumbered Q2 to Q1
Connections:
- net +3.3V: now also Q3.3 (S)
- net GND: now also J3.12, J3.18, J3.3, J3.6, J3.9, J3.MP1, J3.MP2, R13.2, R14.2, U4.12 (GND), U4.2 (GND), U4.25 (GND), U4.3 (GND), U4.30 (GND), U4.31 (GND)
- net VBUS: now also J2.A4 (VBUS), J2.A9 (VBUS), J2.B4 (VBUS), J2.B9 (VBUS), U4.1 (VBUS)
- net PowerButton: now reaches R5.1, SW1.1, U3.1 (PA2)
- net Wii_SHUTDOWN: now reaches U3.10 (PB4)
- net Wii_SHUTDOWN: now also TP7.1
- net Wii_POWER: now reaches U3.11 (PB3)
- net Wii_POWER: now also TP6.1
- net 1.8V_EN: now reaches U3.2 (PA3)
- net 1.8V_EN: now also Q2.2 (G), R13.1
- net 3.3V_EN: now reaches U3.5 (PA4)
- net 3.3V_EN: now also Q3.2 (G), R14.1
- net melon_HPD: now reaches U3.6 (PA5)
- net melon_HPD: now also U4.26 (HPD)
- new net: J2.A1 (GND), J2.A12 (GND), J2.B1 (GND), J2.B12 (GND), J2.S1 (SHIELD)
- new net: J3.16, R11.2
- new net: J3.17, R12.2
- new net +1V8: Q2.3 (S), TP8.1
- new net +5V: J3.19, R11.1, R12.1
- new net 1.8V_Fuji: Q2.1 (D), TP9.1
- new net 3.3V_Fuji: Q3.1 (D), TP10.1
- new net TMDS0+: J3.8, U4.7 (TMDS0-)
- new net TMDS0-: J3.10, U4.6 (TMDS0-)
- new net TMDS1+: J3.5, U4.9 (TMDS1+)
- new net TMDS1-: J3.7, U4.8 (TMDS1-)
- new net TMDS2+: J3.2, U4.11 (TMDS2+)
- new net TMDS2-: J3.4, U4.10 (TMDS2-)
- new net TMDSClk+: J3.11, U4.5 (TMDSCLK+)
- new net TMDSClk-: J3.13, U4.4 (TMDSCLK-)
- new net USB_CC1: J2.A5 (CC1), U4.14 (CC1)
- new net USB_CC2: J2.B5 (CC2), U4.13 (CC1)
- new net USB_RX1+: J2.B11 (RX1+), U4.24 (RX1+)
- new net USB_RX1-: J2.B10 (RX1-), U4.23 (RX1-)
- new net USB_RX2+: J2.A11 (RX2+), U4.22 (RX2+)
- new net USB_RX2-: J2.A10 (RX2-), U4.21 (RX2-)
- new net USB_SBU1: J2.A8 (SBU1), U4.15 (AUX+)
- new net USB_SBU2: J2.B8 (SBU2), U4.16 (AUX-)
- new net USB_TX1+: J2.A2 (TX1+), U4.19 (TX1+)
- new net USB_TX1-: J2.A3 (TX1-), U4.20 (TX1-)
- new net USB_TX2+: J2.B2 (TX2+), U4.17 (TX2+)
- new net USB_TX2-: J2.B3 (TX2-), U4.18 (TX2-)
- new net melonHD_3.3V: U4.27 (SEL0), U4.29 (3.3V_OUT)
- no-connect marks 7 -> 15
Other:
- note added: "HDMI Pin 1"
- note added: "HDMI Pin 19"
- note added: "Note: check footprint"
- moved on the sheet: R5

Commit message: Misc suffering
Parts:
- added U5, U6: ESD204DQAR-ES, Package_DFN_QFN:Diodes_UDFN-10_1.0x2.5mm_P0.5mm, symbol Power_Protection:D3V3XA4B10LP
- J2: footprint Connector_USB:USB_C_Receptacle_Amphenol_12401548E4-2A -> Stormbreaker:GCT_USB4080-03-A_REVA1
- SW1: footprint Button_Switch_THT:SW_Tactile_SPST_Angled_PTS645Vx39-2LFS -> Button_Switch_SMD:Panasonic_EVQPUK_EVQPUB; Mouser (none) -> https://au.mouser.com/ProductDetail/Panasonic/EVQ-P4KB3Q?qs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
Connections:
- net GND: now also J2.A1 (GND), J2.A12 (GND), J2.B1 (GND), J2.B12 (GND), J2.S1 (SHIELD), U5.3 (VSS), U5.8 (VSS), U6.3 (VSS), U6.8 (VSS)
- net TMDS0+: now also U6.1, U6.10 (NC)
- net TMDS0-: now also U6.2, U6.9 (NC)
- net TMDS1+: now also U5.4, U5.7 (NC)
- net TMDS1-: now also U5.5, U5.6 (NC)
- net TMDS2+: now also U5.1, U5.10 (NC)
- net TMDS2-: now also U5.2, U5.9 (NC)
- net TMDSClk+: now also U6.4, U6.7 (NC)
- net TMDSClk-: now also U6.5, U6.6 (NC)
- net USB_SBU1 renamed USB_SBU+
- net USB_SBU2 renamed USB_SBU-
Other:
- note added: "HDMI ESD Suppression"

Commit message: aaaaaaaaaaaa
Parts:
- L1: footprint (none) -> Inductor_SMD:L_Vishay_IHLP-2020; Mouser (none) -> https://au.mouser.com/ProductDetail/Vishay-Dale/IHLP2020CZE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
- Q1, Q2, Q3: footprint (none) -> Package_SO:Vishay_PowerPAK_1212-8_Single; Mouser (none) -> au.mouser.com/ProductDetail/Vishay-Semiconductors/SISS61DN-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
- TP5: footprint (none) -> TestPoint:TestPoint_Pad_D2.0mm
Connections:
- net +1V8: now also Q2.1 (S), Q2.2 (S)
- net +3.3V: now also Q3.1 (S), Q3.2 (S)
- net 1.8V_EN: now also Q2.4 (G); no longer Q2.2 (G)
- net 1.8V_Fuji: now also Q2.5 (D); no longer Q2.1 (D)
- net 3.3V_EN: now also Q3.4 (G); no longer Q3.2 (G)
- net 3.3V_Fuji: now also Q3.5 (D); no longer Q3.1 (D)
- net VCC: now also Q1.1 (S), Q1.2 (S)
- net VDD: now also Q1.5 (D); no longer Q1.1 (D)
- net at R8.1, U3.20 (PA1): now also Q1.4 (G); no longer Q1.2 (G)

Commit message: Mostly done, I think...?
Parts:
- removed D1: LED, symbol Device:LED
- removed R11, R12: 10k, Resistor_SMD:R_0402_1005Metric, symbol Device:R_Small
- removed R4: 4.7k, Resistor_SMD:R_0603_1608Metric, symbol Device:R_Small
- removed R6, R7: 10k, Resistor_SMD:R_0603_1608Metric, symbol Device:R_Small
- TP10: value 3V3_OUT -> 3V3
- TP6: value POWER -> PWR; footprint TestPoint:TestPoint_Pad_D1.5mm -> TestPoint:TestPoint_Pad_D1.0mm
- TP7: value SHUTDOWN -> SHUT; footprint TestPoint:TestPoint_Pad_D1.5mm -> TestPoint:TestPoint_Pad_D1.0mm
- TP9: value 1V8_OUT -> 1V8
Connections:
- no-connect marks 15 -> 17

Commit message: Simplifying, starting from scratch, removing melon
Parts:
- removed J2: USB_C_Receptacle, Stormbreaker:GCT_USB4080-03-A_REVA1, symbol Connector:USB_C_Receptacle
- removed J3: 505278-1933, Stormbreaker:5052781933, symbol SamacSys_Parts:505278-1933
- removed Q2, Q3: PMOS, Package_SO:Vishay_PowerPAK_1212-8_Single, symbol Simulation_SPICE:PMOS
- removed R13, R14: 100k, Resistor_SMD:R_0603_1608Metric, symbol Device:R_Small
- removed TP10: 3V3, TestPoint:TestPoint_Pad_D1.5mm, symbol Connector:TestPoint
- removed U4: ~, Stormbreaker:melonHD_SMT, symbol melonHD_module:melonHD_SMT
- removed U5, U6: ESD204DQAR-ES, Package_DFN_QFN:Diodes_UDFN-10_1.0x2.5mm_P0.5mm, symbol Power_Protection:D3V3XA4B10LP
- added J2: USB_C_Receptacle_USB2.0_14P, Connector_USB:USB_C_Receptacle_Amphenol_12401548E4-2A, symbol Connector:USB_C_Receptacle_USB2.0_14P
- added Q2: NMOS, symbol Simulation_SPICE:NMOS
- added R4, R6: 5.1k, Resistor_SMD:R_0603_1608Metric, symbol Device:R_Small
- TP1, TP2: footprint TestPoint:TestPoint_Pad_D1.5mm -> TestPoint:TestPoint_Pad_D1.0mm
- TP8: value 1V8_IN -> SDA; footprint TestPoint:TestPoint_Pad_D1.5mm -> TestPoint:TestPoint_Pad_D1.0mm
- TP9: value 1V8 -> SCL; footprint TestPoint:TestPoint_Pad_D1.5mm -> TestPoint:TestPoint_Pad_D1.0mm
Connections:
- net +1V8 is gone; now on net SDA: TP8.1
- net 1.8V_Fuji is gone; now on net SCL: TP9.1
- net GND: now also J2.A1 (GND), J2.A12 (GND), J2.B1 (GND), J2.B12 (GND), J2.S1 (SHIELD), Q2.3 (S), R4.1, R6.1
- net VBUS: now also J2.A4 (VBUS), J2.A9 (VBUS), J2.B4 (VBUS), J2.B9 (VBUS)
- net 1.8V_EN: no longer names the net of U3.2 (PA3)
- net 3.3V_EN: no longer names the net of U3.5 (PA4)
- net melon_HPD: no longer names the net of U3.6 (PA5)
- new net: J2.B5 (CC2), R6.2
- new net: J2.A5 (CC1), R4.2
- no-connect marks 17 -> 11
Other:
- note removed: "HDMI ESD Suppression"
- note removed: "HDMI Pin 1"
- note removed: "HDMI Pin 19"
- note removed: "Note: check footprint"

Commit message: hhhhhhhhhh probably going to redesign again
Parts:
- removed Q2: NMOS, symbol Simulation_SPICE:NMOS
- added TP10: VBUS, TestPoint:TestPoint_Pad_D3.0mm, symbol Connector:TestPoint
- added TP11, TP14: BATT, TestPoint:TestPoint_Pad_D3.0mm, symbol Connector:TestPoint
- added TP12, TP15: POWER_BTN, TestPoint:TestPoint_Pad_D1.0mm, symbol Connector:TestPoint
- added TP13: VBUS, TestPoint:TestPoint_Pad_D1.5mm, symbol Connector:TestPoint
- TP4: footprint TestPoint:TestPoint_Pad_D1.5mm -> TestPoint:TestPoint_Pad_D3.0mm
Connections:
- net PowerButton: now also TP12.1, TP15.1
- net VBUS: now also TP10.1, TP13.1
- net BATT: now reaches BT1.1 (+), BT2.1 (+), C2.1, U1.13 (BAT), U1.14 (BAT)
- net BATT: now also TP11.1, TP14.1
Other:
- moved on the sheet: R5
