File: KiCad/Stormbreaker.kicad_sch (KiCad schematic)
At the start: 50 parts, among them J1 Micro_SD_Card_Det2, J2 USB_C_Receptacle_USB2.0_14P, J3 PROG, J4 FAN, J5 I2C, Q1 PMOS, Q2 NMOS, SW1 SW_Push, U1 BQ25895RTW, U3 ATtiny1616-M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

Commit message: More misc improvements
Parts:
- removed J4: FAN, Connector_PinSocket_1.00mm:PinSocket_1x02_P1.00mm_Vertical, symbol Connector_Generic:Conn_01x02
- added TP4: FAN, TestPoint:TestPoint_Pad_D1.0mm, symbol Connector:TestPoint
- C8: footprint Capacitor_SMD:C_0603_1608Metric -> Capacitor_SMD:C_0402_1005Metric
- L1: DigikeyOld (none) -> https://www.digikey.com.au/en/products/detail/susumu/PCMB05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
- R5: footprint Resistor_SMD:R_0603_1608Metric -> Resistor_SMD:R_0402_1005Metric
Connections:
- net GND: now also J1.9 (DET_B); no longer U2.10 (SD_CDZ)
- net at Q2.3 (D): now also TP4.1
- net SD_DECT: now reaches J1.10 (DET_A)
- net SD_DECT: now also U2.10 (SD_CDZ)
- no-connect marks 24 -> 22
Changed lines of the file:
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@@
 	)
 	(junction
-		(at 118.11 177.8)
-		(diameter 0)
-		(color 0 0 0 0)
-	)
-	(junction
 		(at 139.7 90.17)
 		(diameter 0)
@@
 		(color 0 0 0 0)
 	)
+	(junction
+		(at 217.17 137.16)
+		(diameter 0)
+		(color 0 0 0 0)
+	)
 	(no_connect
 		(at 76.2 96.52)
@@
 	)
 	(no_connect
-		(at 229.87 134.62)
-	)
-	(no_connect
 		(at 26.67 57.15)
 	)
@@
 	)
 	(no_connect
-		(at 229.87 137.16)
-	)
-	(no_connect
 		(at 26.67 59.69)
 	)
@@
 	(wire
 		(pts
+			(xy 217.17 137.16) (xy 229.87 137.16)
+		)
+		(stroke
+			(width 0)
+			(type default)
+		)
+	)
+	(wire
+		(pts
 			(xy 143.51 90.17) (xy 143.51 91.44)
 		)
@@
 	(wire
 		(pts
+			(xy 217.17 137.16) (xy 217.17 140.97)
+		)
+		(stroke
+			(width 0)
+			(type default)
+		)
+	)
+	(wire
+		(pts
 			(xy 187.96 95.25) (xy 214.63 95.25)
 		)
@@
 	(wire
 		(pts
-			(xy 118.11 175.26) (xy 113.03 175.26)
-		)
-		(stroke
-			(width 0)
-			(type default)
-		)
-	)
-	(wire
-		(pts
 			(xy 77.47 173.99) (xy 80.01 173.99)
 		)
@@
 	(wire
 		(pts
-			(xy 217.17 127) (xy 217.17 140.97)
+			(xy 217.17 127) (xy 217.17 137.16)
 		)
 		(stroke
@@
 	(wire
 		(pts
-			(xy 118.11 177.8) (xy 118.11 175.26)
-		)
-		(stroke
-			(width 0)
-			(type default)
-		)
-	)
-	(wire
-		(pts
 			(xy 166.37 133.35) (xy 147.32 133.35)
 		)
@@
 		)
 	)
+	(global_label "SD_DECT"
+		(shape input)
+		(at 113.03 175.26 0)
+		(fields_autoplaced yes)
+		(effects
+			(font
+				(size 1.27 1.27)
+			)
+			(justify left)
+		)
+		(property "Intersheetrefs" "${INTERSHEET_REFS}"
+			(at 124.1189 175.26 0)
+			(effects
+				(font
+					(size 1.27 1.27)
+				)
+				(justify left)
+				(hide yes)
+			)
+		)
+	)
 	(global_label "SD_D3"
 		(shape bidirectional)
@@
 		)
 	)
+	(global_label "SD_DECT"
+		(shape output)
+		(at 229.87 134.62 180)
+		(fields_autoplaced yes)
+		(effects
+			(font
+				(size 1.27 1.27)
+			)
+			(justify right)
+		)
+		(property "Intersheetrefs" "${INTERSHEET_REFS}"
+			(at 218.7811 134.62 0)
+			(effects
+				(font
+					(size 1.27 1.27)
+				)
+				(justify right)
+				(hide yes)
+			)
+		)
+	)
 	(global_label "SCL"
 		(shape output)
@@
 	)
 	(global_label "SD_CLK"
-		(shape input)
+		(shape output)
 		(at 116.84 171.45 0)
 		(fields_autoplaced yes)
@@
 		)
 	)
-	(global_label "SDA"
-		(shape bidirectional)
-		(at 116.84 125.73 0)
+	(global_label "SD_DECT"
+		(shape input)
+		(at 156.21 179.07 0)
 		(fields_autoplaced yes)
 		(effects
@@
 		)
 		(property "Intersheetrefs" "${INTERSHEET_REFS}"
-			(at 123.3328 125.73 0)
+			(at 167.2989 179.07 0)
 			(effects
 				(font
@@
 		)
 	)
-	(global_label "SD_D0"
+	(global_label "SDA"
 		(shape bidirectional)
-		(at 229.87 129.54 180)
+		(at 116.84 125.73 0)
 		(fields_autoplaced yes)
 		(effects
@@
 				(size 1.27 1.27)
 			)
-			(justify right)
+			(justify left)
 		)
 		(property "Intersheetrefs" "${INTERSHEET_REFS}"
-			(at 219.8469 129.54 0)
+			(at 123.3328 125.73 0)
 			(effects
 				(font
 					(size 1.27 1.27)
 				)
-				(justify right)
+				(justify left)
 				(hide yes)
 			)
 		)
 	)
-	(symbol
-		(lib_id "Connector_Generic:Conn_01x02")
-		(at 247.65 76.2 0)
-		(unit 1)
-		(exclude_from_sim no)
-		(in_bom yes)
-		(on_board yes)
-		(dnp no)
+	(global_label "SD_D0"
+		(shape bidirectional)
+		(at 229.87 129.54 180)
 		(fields_autoplaced yes)
-		(property "Reference" "J4"
-			(at 250.19 76.1999 0)
-			(effects
-				(font
-					(size 1.27 1.27)
-				)
-				(justify left)
-			)
-		)
-		(property "Value" "FAN"
-			(at 250.19 78.7399 0)
-			(effects
-				(font
-					(size 1.27 1.27)
-				)
-				(justify left)
-			)
-		)
-		(property "Footprint" "Connector_PinSocket_1.00mm:PinSocket_1x02_P1.00mm_Vertical"
-			(at 247.65 76.2 0)
-			(effects
-				(font
-					(size 1.27 1.27)
-				)
-				(hide yes)
-			)
-		)
-		(property "Datasheet" "~"
-			(at 247.65 76.2 0)
-			(effects
-				(font
-					(size 1.27 1.27)
-				)
-				(hide yes)
+		(effects
+			(font
+				(size 1.27 1.27)
 			)
+			(justify right)
 		)
-		(property "Description" "Generic connector, single row, 01x02, script generated (kicad-library-utils/schlib/autogen/connector/)"
-			(at 247.65 76.2 0)
+		(property "Intersheetrefs" "${INTERSHEET_REFS}"
+			(at 219.8469 129.54 0)
 			(effects
 				(font
 					(size 1.27 1.27)
 				)
+				(justify right)
 				(hide yes)
 			)
 		)
-		(pin "2"
-		)
-		(pin "1"
-		)
-		(instances
-			(project ""
-				(path "/dcc89f95-4ae4-4756-aa81-33bf4d3c86ca"
-					(reference "J4")
-					(unit 1)
-				)
-			)
-		)
 	)
 	(symbol
@@
 			)
 		)
-		(property "Footprint" "Capacitor_SMD:C_0603_1608Metric"
+		(property "Footprint" "Capacitor_SMD:C_0402_1005Metric"
 			(at 45.72 156.21 0)
 			(effects
@@
 	)
 	(symbol
-		(lib_id "power:VCC")
-		(at 242.57 76.2 0)
-		(unit 1)
-		(exclude_from_sim no)
-		(in_bom yes)
-		(on_board yes)
-		(dnp no)
-		(fields_autoplaced yes)
-		(property "Reference" "#PWR029"
-			(at 242.57 80.01 0)
-			(effects
-				(font
-					(size 1.27 1.27)
-				)
-				(hide yes)
-			)
-		)
-		(property "Value" "VCC"
-			(at 242.57 71.12 0)
-			(effects
-				(font
-					(size 1.27 1.27)
-				)
-			)
-		)
-		(property "Footprint" ""
-			(at 242.57 76.2 0)
-			(effects
-				(font
-					(size 1.27 1.27)
-				)
-				(hide yes)
-			)
-		)
-		(property "Datasheet" ""
-			(at 242.57 76.2 0)
-			(effects
-				(font
-					(size 1.27 1.27)
-				)
-				(hide yes)
-			)
-		)
-		(property "Description" "Power symbol creates a global label with name \"VCC\""
-			(at 242.57 76.2 0)
-			(effects
-				(font
-					(size 1.27 1.27)
-				)
-				(hide yes)
-			)
-		)
-		(pin "1"
-		)
-		(instances
-			(project "Stormbreaker"
-				(path "/dcc89f95-4ae4-4756-aa81-33bf4d3c86ca"
-					(reference "#PWR029")
-					(unit 1)
-				)
-			)
-		)
-	)
-	(symbol
 		(lib_id "Device:Battery_Cell")
 		(at 114.3 88.9 0)
@@
 	)
 	(symbol
+		(lib_id "Connector:TestPoint")
+		(at 242.57 78.74 270)
+		(unit 1)
+		(exclude_from_sim no)
+		(in_bom yes)
+		(on_board yes)
+		(dnp no)
+		(fields_autoplaced yes)
+		(property "Reference" "TP4"
+			(at 247.65 77.4699 90)
+			(effects
+				(font
+					(size 1.27 1.27)
+				)
+				(justify left)
+			)
+		)
+		(property "Value" "FAN"
+			(at 247.65 80.0099 90)
+			(effects
+				(font
+					(size 1.27 1.27)
+				)
+				(justify left)
+			)
+		)
+		(property "Footprint" "TestPoint:TestPoint_Pad_D1.0mm"
+			(at 242.57 83.82 0)
+			(effects
+				(font
+					(size 1.27 1.27)
+				)
+				(hide yes)
+			)
+		)
+		(property "Datasheet" "~"
+			(at 242.57 83.82 0)
+			(effects
+				(font
+					(size 1.27 1.27)
+				)
+				(hide yes)
+			)
+		)
+		(property "Description" "test point"
+			(at 242.57 78.74 0)
+			(effects
+				(font
+					(size 1.27 1.27)
+				)
+				(hide yes)
+			)
+		)
+		(pin "1"
+		)
+		(instances
+			(project "Stormbreaker"
+				(path "/dcc89f95-4ae4-4756-aa81-33bf4d3c86ca"
+					(reference "TP4")
+					(unit 1)
+				)
+			)
+		)
+	)
+	(symbol
 		(lib_id "Device:C_Small")
 		(at 71.12 68.58 0)
@@
 			)
 		)
-		(property "Footprint" "Resistor_SMD:R_0603_1608Metric"
+		(property "Footprint" "Resistor_SMD:R_0402_1005Metric"
 			(at 207.01 66.04 0)
 			(effects
@@
 			(at 104.14 71.12 90)
 			(effects
+				(font
+					(size 1.27 1.27)
+				)
+				(hide yes)
+			)
+		)
+		(property "DigikeyOld" "https://www.digikey.com.au/en/products/detail/susumu/PCMB053T-3R3MS/3672034?s=N4IgTCBcDaICwAYAcBaAjAVjA9KByAIiALoC%2BQA"
+			(at 104.14 71.12 90)
+			(effects

Commit message: More more misc improvements
Parts:
- removed TP8: VCC, TestPoint:TestPoint_Pad_D2.0mm, symbol Connector:TestPoint
- added C16: 10uF, Capacitor_SMD:C_0603_1608Metric, symbol Device:C_Small
- C5, C6: footprint Capacitor_SMD:C_0603_1608Metric -> Capacitor_SMD:C_0402_1005Metric
- TP5: footprint TestPoint:TestPoint_Pad_D2.0mm -> TestPoint:TestPoint_Pad_D2.5mm
Connections:
- net BATT: now also C16.1
- net GND: now also C16.2
Other:
- moved on the sheet: R10, R9
