File: KiCad/cafebara.kicad_sch (KiCad schematic)
At the start: 27 parts, among them J1 Micro_SD_Card_Det2, J2 USB_C_Receptacle_USB2.0_14P, J3 PROG, J4 505278-1933, J5 I2C, Q1 NMOS, SW1 SW_Push, U3 ATtiny1616-M

Commit message: Minor misc updates
Parts:
- added TP6: HPD, TestPoint:TestPoint_Pad_D1.5mm, symbol Connector:TestPoint
Connections:
- net HPD: now also TP6.1
Other:
- moved on the sheet: Q1, TP4
Changed lines of the file:
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@@
 	)
 	(junction
+		(at 85.09 110.49)
+		(diameter 0)
+		(color 0 0 0 0)
+	)
+	(junction
 		(at 77.47 173.99)
 		(diameter 0)
@@
 	(wire
 		(pts
+			(xy 219.71 71.12) (xy 217.17 71.12)
+		)
+		(stroke
+			(width 0)
+			(type default)
+		)
+	)
+	(wire
+		(pts
 			(xy 330.2 140.97) (xy 334.01 140.97)
 		)
@@
 	(wire
 		(pts
+			(xy 85.09 110.49) (xy 99.06 110.49)
+		)
+		(stroke
+			(width 0)
+			(type default)
+		)
+	)
+	(wire
+		(pts
 			(xy 317.5 123.19) (xy 334.01 123.19)
 		)
@@
 	(wire
 		(pts
+			(xy 77.47 110.49) (xy 85.09 110.49)
+		)
+		(stroke
+			(width 0)
+			(type default)
+		)
+	)
+	(wire
+		(pts
 			(xy 116.84 163.83) (xy 113.03 163.83)
 		)
@@
 	(global_label "FAN_PWM"
 		(shape output)
-		(at 217.17 71.12 0)
+		(at 219.71 71.12 0)
 		(fields_autoplaced yes)
 		(effects
@@
 		)
 		(property "Intersheetrefs" "${INTERSHEET_REFS}"
-			(at 228.8033 71.12 0)
+			(at 231.3433 71.12 0)
 			(effects
 				(font
@@
 	(global_label "HPD"
 		(shape output)
-		(at 99.06 110.49 180)
+		(at 77.47 110.49 180)
 		(fields_autoplaced yes)
 		(effects
@@
 		)
 		(property "Intersheetrefs" "${INTERSHEET_REFS}"
-			(at 92.2043 110.49 0)
+			(at 70.6143 110.49 0)
 			(effects
 				(font
@@
 	(global_label "FAN_PWM"
 		(shape input)
-		(at 259.08 58.42 180)
+		(at 269.24 60.96 180)
 		(fields_autoplaced yes)
 		(effects
@@
 		)
 		(property "Intersheetrefs" "${INTERSHEET_REFS}"
-			(at 247.4467 58.42 0)
+			(at 257.6067 60.96 0)
 			(effects
 				(font
@@
 	(symbol
 		(lib_id "Connector:TestPoint")
-		(at 266.7 53.34 0)
+		(at 276.86 55.88 0)
 		(unit 1)
 		(exclude_from_sim no)
@@
 		(fields_autoplaced yes)
 		(property "Reference" "TP4"
-			(at 269.24 48.7679 0)
+			(at 279.4 51.3079 0)
 			(effects
 				(font
@@
 		)
 		(property "Value" "FAN"
-			(at 269.24 51.3079 0)
+			(at 279.4 53.8479 0)
 			(effects
 				(font
@@
 		)
 		(property "Footprint" "TestPoint:TestPoint_Pad_D1.5mm"
-			(at 271.78 53.34 0)
+			(at 281.94 55.88 0)
 			(effects
 				(font
@@
 		)
 		(property "Datasheet" "~"
-			(at 271.78 53.34 0)
+			(at 281.94 55.88 0)
 			(effects
 				(font
@@
 		)
 		(property "Description" "test point"
-			(at 266.7 53.34 0)
+			(at 276.86 55.88 0)
 			(effects
 				(font
@@
 	(symbol
 		(lib_id "Simulation_SPICE:NMOS")
-		(at 264.16 58.42 0)
+		(at 274.32 60.96 0)
 		(unit 1)
 		(exclude_from_sim no)
@@
 		(fields_autoplaced yes)
 		(property "Reference" "Q1"
-			(at 270.51 57.1499 0)
+			(at 280.67 59.6899 0)
 			(effects
 				(font
@@
 		)
 		(property "Value" "NMOS"
-			(at 270.51 59.6899 0)
+			(at 280.67 62.2299 0)
 			(effects
 				(font
@@
 		)
 		(property "Footprint" "Package_TO_SOT_SMD:SOT-523"
-			(at 269.24 55.88 0)
+			(at 279.4 58.42 0)
 			(effects
 				(font
@@
 		)
 		(property "Datasheet" "https://ngspice.sourceforge.io/docs/ngspice-html-manual/manual.xhtml#cha_MOSFETs"
-			(at 264.16 71.12 0)
+			(at 274.32 73.66 0)
 			(effects
 				(font
@@
 		)
 		(property "Description" "N-MOSFET transistor, drain/source/gate"
-			(at 264.16 58.42 0)
+			(at 274.32 60.96 0)
 			(effects
 				(font
@@
 		)
 		(property "Sim.Device" "NMOS"
-			(at 264.16 75.565 0)
+			(at 274.32 78.105 0)
 			(effects
 				(font
@@
 		)
 		(property "Sim.Type" "VDMOS"
-			(at 264.16 77.47 0)
+			(at 274.32 80.01 0)
 			(effects
 				(font
@@
 		)
 		(property "Sim.Pins" "1=D 2=G 3=S"
-			(at 264.16 73.66 0)
+			(at 274.32 76.2 0)
 			(effects
 				(font
@@
 		)
 		(property "MouserOld" "https://au.mouser.com/ProductDetail/Diodes-Incorporated/DMN2310U-7?qs=xZ%2FP%252Ba9zWqY%252BAdKLxIytvQ%3D%3D"
-			(at 264.16 58.42 0)
+			(at 274.32 60.96 0)
 			(effects
 				(font
@@
 		)
 		(property "Digikey" "https://www.digikey.com.au/en/products/detail/good-ark-semiconductor/SSF2320Y/18667769"
-			(at 264.16 58.42 0)
+			(at 274.32 60.96 0)
 			(effects
 				(font
@@
 	(symbol
 		(lib_id "power:GND")
-		(at 266.7 63.5 0)
+		(at 276.86 66.04 0)
 		(unit 1)
 		(exclude_from_sim no)
@@
 		(fields_autoplaced yes)
 		(property "Reference" "#PWR028"
-			(at 266.7 69.85 0)
+			(at 276.86 72.39 0)
 			(effects
 				(font
@@
 		)
 		(property "Value" "GND"
-			(at 266.7 68.58 0)
+			(at 276.86 71.12 0)
 			(effects
 				(font
@@
 		)
 		(property "Footprint" ""
-			(at 266.7 63.5 0)
+			(at 276.86 66.04 0)
 			(effects
 				(font
@@
 		)
 		(property "Datasheet" ""
-			(at 266.7 63.5 0)
+			(at 276.86 66.04 0)
 			(effects
 				(font
@@
 		)
 		(property "Description" "Power symbol creates a global label with name \"GND\" , ground"
-			(at 266.7 63.5 0)
+			(at 276.86 66.04 0)
 			(effects
 				(font
@@
 					(unit 1)
 				)
+			)
+		)
+	)
+	(symbol
+		(lib_id "Connector:TestPoint")
+		(at 85.09 110.49 0)
+		(unit 1)
+		(exclude_from_sim no)
+		(in_bom yes)
+		(on_board yes)
+		(dnp no)
+		(property "Reference" "TP6"
+			(at 82.55 108.4581 0)
+			(effects
+				(font
+					(size 1.27 1.27)
+				)
+				(justify right)
+			)
+		)
+		(property "Value" "HPD"
+			(at 82.55 105.9181 0)
+			(effects
+				(font
+					(size 1.27 1.27)
+				)
+				(justify right)
+			)
+		)
+		(property "Footprint" "TestPoint:TestPoint_Pad_D1.5mm"
+			(at 90.17 110.49 0)
+			(effects
+				(font
+					(size 1.27 1.27)
+				)
+				(hide yes)
+			)
+		)
+		(property "Datasheet" "~"
+			(at 90.17 110.49 0)
+			(effects
+				(font
+					(size 1.27 1.27)
+				)
+				(hide yes)
+			)
+		)
+		(property "Description" "test point"
+			(at 85.09 110.49 0)
+			(effects
+				(font
+					(size 1.27 1.27)
+				)
+				(hide yes)
+			)
+		)
+		(pin "1"
+		)
+		(instances
+			(project "cafebara"
+				(path "/dcc89f95-4ae4-4756-aa81-33bf4d3c86ca"
+					(reference "TP6")
+					(unit 1)
+				)

Commit message: Misc changes to cafebara, add temperature board
Parts:
- removed J4: 505278-1933, Connector_FFC-FPC:TE_1-1734839-9_1x19-1MP_P0.5mm_Horizontal, symbol SamacSys_Parts:505278-1933
- added J4: Conn_01x19_MountingPin, Connector_FFC-FPC:TE_1-1734839-9_1x19-1MP_P0.5mm_Horizontal, symbol Connector_Generic_MountingPin:Conn_01x19_MountingPin
Connections:
- net +5V: now also J4.2 (Pin_2)
- net GND: now also J4.12 (Pin_12), J4.15 (Pin_15), J4.18 (Pin_18), J4.3 (Pin_3), J4.9 (Pin_9), J4.MP (MountPin)
- net HDMI_SCL: now also J4.5 (Pin_5)
- net HDMI_SDA: now also J4.4 (Pin_4)
- net HPD: now also J4.1 (Pin_1)
- net TMDS0+: now also J4.13 (Pin_13)
- net TMDS0-: now also J4.11 (Pin_11)
- net TMDS1+: now also J4.16 (Pin_16)
- net TMDS1-: now also J4.14 (Pin_14)
- net TMDS2+: now also J4.19 (Pin_19)
- net TMDS2-: now also J4.17 (Pin_17)
- net TMDSClk+: now also J4.10 (Pin_10)
- net TMDSClk-: now also J4.8 (Pin_8)
Other:
- note removed: "HDMI Pin 1"
- note removed: "HDMI Pin 19"

Commit message: Add alert pin, EDID EEPROM, misc other changes
Parts:
- added C7: 10uF, Capacitor_SMD:C_0603_1608Metric, symbol Device:C_Small
- added J6: EDID, cafebara:UPDI Pads, symbol Connector_Generic:Conn_01x03
- added TP7: ALERT, cafebara:TestPoint_Pad_D1.0mm_Small, symbol Connector:TestPoint
- added U4: M24C02-WMN, Package_SO:SOIC-8_3.9x4.9mm_P1.27mm, symbol Memory_EEPROM:M24C02-WMN
- J3: footprint Stormbreaker:UPDI Pads -> cafebara:UPDI Pads
Connections:
- net +5V: now also C7.1, U4.8 (VCC)
- net GND: now also C7.2, U4.1 (E0), U4.2 (E1), U4.3 (E2), U4.4 (VSS)
- net HDMI_SCL: now also J6.2 (Pin_2), U4.6 (SCL)
- net HDMI_SDA: now also J6.1 (Pin_1), U4.5 (SDA)
- net ~{ALERT}: now reaches U3.11 (PB3)
- net ~{ALERT}: now also TP7.1
- new net EEPROM_~{WC}: J6.3 (Pin_3), U4.7 (~{WC})
- no-connect marks 15 -> 14
Other:
- note added: "Sets address to 0x50 for EDID"
- moved on the sheet: J4

Commit message: Possibly planning to enlarge board...
Parts:
- added H1, H2, H3, H4: GND, TestPoint_Plated_Hole_D2.0mm, symbol Mechanical:MountingHole_Pad
Connections:
- net GND: now also H1.1, H2.1, H3.1, H4.1

Commit message: Expand board, add charge IC, other misc changes
Parts:
- added BT1: Battery_Cell, symbol Device:Battery_Cell
- added C10, C11: 10uF, Capacitor_SMD:C_0402_1005Metric, symbol Device:C_Small
- added C12: 47nF, Capacitor_SMD:C_0402_1005Metric, symbol Device:C_Small
- added C13, C15, C16, C9: 10uF, Capacitor_SMD:C_0603_1608Metric, symbol Device:C_Small
- added C14: 4.7uF, Capacitor_SMD:C_0402_1005Metric, symbol Device:C_Small
- added C8: 22uF, Capacitor_SMD:C_0402_1005Metric, symbol Device:C_Small
- added L1: 3.3uH, Inductor_SMD:L_APV_APH0420, symbol Device:L_Small
- added R6: 260, Resistor_SMD:R_0402_1005Metric, symbol Device:R_Small
- added R7: 5.23k, Resistor_SMD:R_0402_1005Metric, symbol Device:R_Small
- added R8: 30.1k, Resistor_SMD:R_0402_1005Metric, symbol Device:R_Small
- added TP11: 5V, TestPoint:TestPoint_Pad_D1.5mm, symbol Connector:TestPoint
- added TP8: VCC, TestPoint:TestPoint_Plated_Hole_D2.0mm, symbol Connector:TestPoint
- added TP9: GND, TestPoint:TestPoint_Plated_Hole_D2.0mm, symbol Connector:TestPoint
- added U5: BQ25895RTW, Package_DFN_QFN:Texas_RTW_WQFN-24-1EP_4x4mm_P0.5mm_EP2.7x2.7mm_ThermalVias, symbol Battery_Management:BQ25895RTW
- TP5: value BQ -> BATT; footprint cafebara:TestPoint_Pad_D1.0mm_Small -> TestPoint:TestPoint_Plated_Hole_D2.0mm
- U4: Digikey (none) -> https://www.digikey.com.au/en/products/detail/stmicroelectr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
Connections:
- net +3.3V_LDO: no longer U1.27 (SEL0)
- net +5V: now also TP11.1
- net BQ_STAT: now also U5.4 (STAT); no longer TP5.1, U3.15 (PC0)
- net GND: now also U1.27 (SEL0), BT1.2 (-), C10.2, C11.2, C13.2, C14.1, C15.2, C16.2, C8.1, C9.2, R6.1, R8.1, TP9.1, U5.17 (PGND), U5.18 (PGND), U5.25 (PGND), U5.9 (~{CE})
- net SCL: now also U5.5 (SCL)
- net SDA: now also U5.6 (SDA)
- net VBUS: now also C15.1, C9.1, U5.1 (VBUS)
- net VCC: now also C10.1, C11.1, L1.2, TP8.1, U5.15 (SYS), U5.16 (SYS)
- new net: R6.2, U5.10 (ILIM)
- new net: R7.1, R8.2, U5.11 (TS)
- new net: C12.1, L1.1, U5.19 (SW), U5.20 (SW)
- new net: C12.2, U5.21 (BTST)
- new net: C14.2, R7.2, U5.22 (REGN)
- new net: C8.2, U5.23 (PMID)
- new net BATT: BT1.1 (+), C13.1, C16.1, TP5.1, U5.13 (BAT), U5.14 (BAT)
- new net ~{INT}: U3.15 (PC0), U5.7 (INT)
- no-connect marks 14 -> 19
