File: HDMI_Mux/HDMI_Mux.kicad_sch (KiCad schematic)
At the start: 12 parts, among them J1 505278-1933, J2 Conn_01x19_MountingPin, J3 Conn_01x19_MountingPin, U1 TS3DV20812, U2 ESD204DQAR-ES, U3 ESD204DQAR-ES, U4 ESD204DQAR-ES, U5 ESD204DQAR-ES

Commit message: Finish HDMI mux, misc improvements to cafebara
Parts:
- added TP1: +5V, TestPoint:TestPoint_Pad_D2.5mm, symbol Connector:TestPoint
- added TP2: GND, TestPoint:TestPoint_Pad_D2.5mm, symbol Connector:TestPoint
- added TP3: SEL, TestPoint:TestPoint_Pad_D1.5mm, symbol Connector:TestPoint
- J1, J2, J3: footprint Connector_FFC-FPC:TE_1-1734839-9_1x19-1MP_P0.5mm_Horizontal -> Connector_FFC-FPC:Hirose_FH12-19S-0.5SH_1x19-1MP_P0.50mm_Horizontal
- U1: value TS3DV20812 -> TS3DV642; footprint Package_DFN_QFN:Texas_RHH0036C_VQFN-36-1EP_6x6mm_P0.5mm_EP4.4x4.4mm_ThermalVias -> Package_DFN_QFN:WQFN-42-1EP_3.5x9mm_P0.5mm_EP2.05x7.55mm_ThermalVias
Connections:
- net +3.3V is gone; now on net TMDS1_A-: U1.35 (D1_A-)
- net SEL is gone; now on net TMDS1_B+: U1.27 (D1_B+)
- net +5V: now also U1.1 (VCC), U1.16 (SEL1), U1.2 (EN), TP1.1
- net GND: now also U1.43 (GND), TP2.1; no longer U1.11 (GND), U1.37 (GND)
- net HDMI_SCL: now also U1.4 (SDA); no longer U1.12 (A2)
- net HDMI_SDA: now also U1.3 (SCL); no longer U1.4 (A1)
- net HPD: now also U1.14 (HPD); no longer U1.34 (A3)
- net HPD_A: now also U1.19 (HPD_A); no longer U1.33 (A3_A)
- net HPD_B: now also U1.21 (HPD_B); no longer U1.32 (A3_B)
- net SCL_A: now also U1.41 (SDA_A); no longer U1.13 (A2_A)
- net SCL_B: now also U1.39 (SDA_B); no longer U1.14 (A2_B)
- net SDA_A: now also U1.42 (SCL_A); no longer U1.5 (A1_A)
- net SDA_B: now also U1.40 (SCL_B); no longer U1.6 (A1_B)
- net TMDS0+: now also U1.10 (D2+); no longer U1.7 (D2+)
- net TMDS0-: now also U1.11 (D2-); no longer U1.8 (D2-)
- net TMDS0_A+: now also U1.34 (D2_A+); no longer U1.22 (D2_A+)
- net TMDS0_A-: now also U1.33 (D2_A-); no longer U1.21 (D2_A-)
- net TMDS0_B+: now also U1.25 (D2_B+); no longer U1.20 (D2_B+)
- net TMDS0_B-: now also U1.24 (D2_B-); no longer U1.19 (D2_B-)
- net TMDS1+: now also U1.7 (D1+); no longer U1.2 (D1+)
- net TMDS1-: now also U1.8 (D1-); no longer U1.3 (D1-)
- net TMDS1_A+: now also U1.36 (D1_A+); no longer U1.26 (D1_A+)
- net TMDS1_A-: no longer U1.25 (D1_A-)
- net TMDS1_B+: no longer U1.24 (D1_B+)
- net TMDS1_B-: now also U1.26 (D1_B-); no longer U1.23 (D1_B-)
- net TMDS2+: now also U1.5 (D0+); no longer U1.36 (D0+)
- net TMDS2-: now also U1.6 (D0-); no longer U1.1 (D0-)
- net TMDS2_A+: now also U1.38 (D0_A+); no longer U1.31 (D0_A+)
- net TMDS2_A-: now also U1.37 (D0_A-); no longer U1.30 (D0_A-)
- net TMDSClk+: now also U1.12 (D3+); no longer U1.9 (D3+)
- net TMDSClk-: now also U1.13 (D3-); no longer U1.10 (D3-)
- net TMDSClk_A+: now also U1.32 (D3_A+); no longer U1.18 (D3_A+)
- net TMDSClk_A-: now also U1.31 (D3_A-); no longer U1.17 (D3_A-)
- net TMDSClk_B+: now also U1.23 (D3_B+); no longer U1.16 (D3_B+)
- net TMDSClk_B-: now also U1.22 (D3_B-); no longer U1.15 (D3_B-)
- new net: U1.30 (NC), U1.9 (NC)
- new net SEL2: TP3.1, U1.17 (SEL2)
- no-connect marks 6 -> 7
