File: Regs/Cafebara_regs.kicad_pcb (KiCad board)
At the start: 4 copper layers, 43.2 x 28.2 mm, 53 parts, among them U1 TDA38826XUMA1, U2 TDA38826XUMA1, U3 FAN49100AUC330X, U4 TLV74311PDBVR, U5 AP2210K-ADJ, U6 TPS61232DRC

Commit message: Other misc reg changes
Parts:
- added C31: 100uF, Capacitor_Tantalum_SMD:CP_EIA-3216-10_Kemet-I, F.Cu at (135.0, 122.8)
- added R12: 10k, Resistor_SMD:R_0402_1005Metric, F.Cu at (99.8, 118.8)
- C1, C10: footprint Capacitor_SMD:C_0805_2012Metric -> Capacitor_SMD:C_0603_1608Metric
- C11, C2: value 47uF -> 100uF; footprint Capacitor_SMD:C_0805_2012Metric -> Capacitor_Tantalum_SMD:CP_EIA-3216-10_Kemet-I
- moved C12 4.25 mm to (119.5, 115.8)
- moved C3 4.25 mm to (107.2, 115.8)
- moved C11 0.56 mm to (119.8, 112.5)
- moved C2 0.56 mm to (107.5, 112.5)
- moved C1 0.50 mm to (107.2, 114.5)
- moved C10 0.50 mm to (119.5, 114.5)
- moved C19 0.50 mm to (114.8, 116.8)
- moved C16 0.25 mm to (115.5, 120.0)
- moved C7 0.25 mm to (103.2, 120.0)
- moved L3 0.25 mm to (111.0, 114.0)
Routing:
- net VCC: vias 120 -> 117
- net GND: vias 152 -> 154

Commit message: misc changes and improvements
Parts:
- added TP2: +1V, TestPoint:TestPoint_THTPad_D2.5mm_Drill1.2mm, F.Cu at (104.5, 132.0)
- added TP3: +1.15V, TestPoint:TestPoint_THTPad_D2.5mm_Drill1.2mm, F.Cu at (120.2, 132.0)
- added TP4: +5V, TestPoint:TestPoint_THTPad_D2.5mm_Drill1.2mm, F.Cu at (135.0, 117.2)
- added TP5: GND, TestPoint:TestPoint_THTPad_D2.5mm_Drill1.2mm, F.Cu at (121.8, 109.0)
- added TP6: VCC, TestPoint:TestPoint_THTPad_D2.5mm_Drill1.2mm, F.Cu at (103.0, 109.2)
Routing:
- net Net-(L4-Pad2): vias 19 -> 31
- net GND: vias 154 -> 143
- net +5V: vias 34 -> 22
- net +1V15: vias 85 -> 75
- net +1V0: vias 85 -> 75
Other:
- board text added: "+1.1 5V"
- board text added: "+1.1 V"
- board text removed: "+1.15V"
- board text removed: "+1.1V"
