File: Regs/Cafebara_regs.kicad_sch (KiCad schematic)
At the start: 55 parts, among them U1 TDA38826XUMA1, U2 TDA38826XUMA1, U3 FAN49100AUC330X, U4 TLV74311PDBVR, U5 AP2210K-ADJ, U6 TPS61232DRC

Commit message: Largely finish positioning and routing
Parts:
- removed TP2, TP3: GND, TestPoint:TestPoint_Plated_Hole_D2.0mm, symbol Connector:TestPoint
- removed TP4: +1.15V, TestPoint:TestPoint_Plated_Hole_D2.0mm, symbol Connector:TestPoint
- C22, C23, C24, C25: footprint Capacitor_SMD:C_0402_1005Metric -> Capacitor_SMD:C_0603_1608Metric
- TP1: value +1V -> EN; footprint TestPoint:TestPoint_Plated_Hole_D2.0mm -> TestPoint:TestPoint_Pad_D1.5mm
Connections:
- net +1V0: no longer TP1.1
- net EN: now also TP1.1
Other:
- moved on the sheet: TP1

Commit message: Regulator board design finalisation
Parts:
- added H1: ~, MountingHole:MountingHole_2.2mm_M2_Pad_Via, symbol Mechanical:MountingHole_Pad
Connections:
- net GND: now also H1.1
Changed lines of the file:
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@@
+	)
+	(symbol
+		(lib_id "power:GND")
+		(at 180.34 135.89 0)
+		(unit 1)
+		(exclude_from_sim no)
+		(in_bom yes)
+		(on_board yes)
+		(dnp no)
+		(fields_autoplaced yes)
+		(property "Reference" "#PWR03"
+			(at 180.34 142.24 0)
+			(effects
+				(font
+					(size 1.27 1.27)
+				)
+				(hide yes)
+			)
+		)
+		(property "Value" "GND"
+			(at 180.34 140.97 0)
+			(effects
+				(font
+					(size 1.27 1.27)
+				)
+			)
+		)
+		(property "Footprint" ""
+			(at 180.34 135.89 0)
+			(effects
+				(font
+					(size 1.27 1.27)
+				)
+				(hide yes)
+			)
+		)
+		(property "Datasheet" ""
+			(at 180.34 135.89 0)
+			(effects
+				(font
+					(size 1.27 1.27)
+				)
+				(hide yes)
+			)
+		)
+		(property "Description" "Power symbol creates a global label with name \"GND\" , ground"
+			(at 180.34 135.89 0)
+			(effects
+				(font
+					(size 1.27 1.27)
+				)
+				(hide yes)
+			)
+		)
+		(pin "1"
+		)
+		(instances
+			(project "Cafebara_regs"
+				(path "/f90fb1fb-a242-4f20-8a51-2c53666311a4"
+					(reference "#PWR03")
+					(unit 1)
+				)
+			)
+		)
 	)
 	(symbol
@@
 					(unit 1)
 				)
+			)
+		)
+	)
+	(symbol
+		(lib_id "Mechanical:MountingHole_Pad")
+		(at 180.34 133.35 0)
+		(unit 1)
+		(exclude_from_sim yes)
+		(in_bom no)
+		(on_board yes)
+		(dnp no)
+		(fields_autoplaced yes)
+		(property "Reference" "H1"
+			(at 182.88 130.8099 0)
+			(effects
+				(font
+					(size 1.27 1.27)
+				)
+				(justify left)
+			)
+		)
+		(property "Value" "~"
+			(at 182.88 133.3499 0)
+			(effects
+				(font
+					(size 1.27 1.27)
+				)
+				(justify left)
+			)
+		)
+		(property "Footprint" "MountingHole:MountingHole_2.2mm_M2_Pad_Via"
+			(at 180.34 133.35 0)
+			(effects
+				(font
+					(size 1.27 1.27)
+				)
+				(hide yes)
+			)
+		)
+		(property "Datasheet" "~"
+			(at 180.34 133.35 0)
+			(effects
+				(font
+					(size 1.27 1.27)
+				)
+				(hide yes)
+			)
+		)
+		(property "Description" "Mounting Hole with connection"
+			(at 180.34 133.35 0)
+			(effects
+				(font
+					(size 1.27 1.27)
+				)
+				(hide yes)
+			)
+		)
+		(pin "1"
+		)
+		(instances
+			(project ""
+				(path "/f90fb1fb-a242-4f20-8a51-2c53666311a4"
+					(reference "H1")
+					(unit 1)
+				)

Commit message: Other misc reg changes
Parts:
- removed C11, C2: 47uF, Capacitor_SMD:C_0805_2012Metric, symbol Device:C_Small
- added C11, C2, C31: 100uF, Capacitor_Tantalum_SMD:CP_EIA-3216-10_Kemet-I, symbol Device:C_Polarized_Small
- added R12: 10k, Resistor_SMD:R_0402_1005Metric, symbol Device:R_Small
- C1, C10: footprint Capacitor_SMD:C_0805_2012Metric -> Capacitor_SMD:C_0603_1608Metric
Connections:
- net +5V: now also C31.1
- net EN: now also R12.2
- net GND: now also C11.2, C2.2, C31.2, R12.1
- net P_{VIN}: now also C11.1, C2.1

Commit message: misc changes and improvements
Parts:
- added TP2: +1V, TestPoint:TestPoint_THTPad_D2.5mm_Drill1.2mm, symbol Connector:TestPoint
- added TP3: +1.15V, TestPoint:TestPoint_THTPad_D2.5mm_Drill1.2mm, symbol Connector:TestPoint
- added TP4: +5V, TestPoint:TestPoint_THTPad_D2.5mm_Drill1.2mm, symbol Connector:TestPoint
- added TP5: GND, TestPoint:TestPoint_THTPad_D2.5mm_Drill1.2mm, symbol Connector:TestPoint
- added TP6: VCC, TestPoint:TestPoint_THTPad_D2.5mm_Drill1.2mm, symbol Connector:TestPoint
Connections:
- net +1V0: now also TP2.1
- net +1V15: now also TP3.1
- net +5V: now also TP4.1
- net GND: now also TP5.1
- net P_{VIN}: now also TP6.1
Other:
- moved on the sheet: TP1
